File: 23-BSPD-ELC/BMSComparator.kicad_sch (KiCad schematic)
At the start: 16 parts, among them U11 LM239

Commit message: Updated pcb layout; Watchdog on board still in progress
Parts:
- RV10, RV11, RV12, RV9: footprint LHRE Footprint Library:PV36W201C01B00 -> Global Libraries:PVG5A
Changed lines of the file:
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@@
       (effects (font (size 1.27 1.27)) (justify right))
     )
-    (property "Footprint" "LHRE Footprint Library:PV36W201C01B00" (id 2) (at 102.87 138.43 0)
+    (property "Footprint" "Global Libraries:PVG5A" (id 2) (at 102.87 138.43 0)
       (effects (font (size 1.27 1.27)) hide)
     )
@@
       (effects (font (size 1.27 1.27)) (justify right))
     )
-    (property "Footprint" "LHRE Footprint Library:PV36W201C01B00" (id 2) (at 104.14 113.03 0)
+    (property "Footprint" "Global Libraries:PVG5A" (id 2) (at 104.14 113.03 0)
       (effects (font (size 1.27 1.27)) hide)
     )
@@
       (effects (font (size 1.27 1.27)) (justify right))
     )
-    (property "Footprint" "LHRE Footprint Library:PV36W201C01B00" (id 2) (at 102.87 74.93 0)
+    (property "Footprint" "Global Libraries:PVG5A" (id 2) (at 102.87 74.93 0)
       (effects (font (size 1.27 1.27)) hide)
     )
@@
       (effects (font (size 1.27 1.27)) (justify right))
     )
-    (property "Footprint" "LHRE Footprint Library:PV36W201C01B00" (id 2) (at 102.87 48.26 0)
-      (effects (font (size 1.27 1.27)) hide)
-    )
+    (property "Footprint" "Global Libraries:PVG5A" (id 2) (at 102.87 48.26 0)
+      (effects (font (size 1.27 1.27)) hide)
+    )
