File: 23-BSPD-ELC/BrakeComparator.kicad_sch (KiCad schematic)
At the start: 16 parts, among them U10 LM239, U9 LM239

Commit message: Updated pcb layout; Watchdog on board still in progress
Parts:
- RV6, RV7, RV8: footprint LHRE Footprint Library:PV36W201C01B00 -> Global Libraries:PVG5A
Changed lines of the file:
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@@
       (effects (font (size 1.27 1.27)) (justify right))
     )
-    (property "Footprint" "LHRE Footprint Library:PV36W201C01B00" (id 2) (at 99.06 46.99 0)
+    (property "Footprint" "Global Libraries:PVG5A" (id 2) (at 99.06 46.99 0)
       (effects (font (size 1.27 1.27)) hide)
     )
-    (property "Datasheet" "https://www.mouser.com/datasheet/2/54/pv36-907345.pdf" (id 3) (at 99.06 46.99 0)
+    (property "Datasheet" "https://www.mouser.com/datasheet/2/54/pvg5-907351.pdf" (id 3) (at 99.06 46.99 0)
       (effects (font (size 1.27 1.27)) hide)
     )
@@
       (effects (font (size 1.27 1.27)) (justify right))
     )
-    (property "Footprint" "LHRE Footprint Library:PV36W201C01B00" (id 2) (at 106.68 77.47 0)
+    (property "Footprint" "Global Libraries:PVG5A" (id 2) (at 106.68 77.47 0)
       (effects (font (size 1.27 1.27)) hide)
     )
-    (property "Datasheet" "https://www.mouser.com/datasheet/2/54/pv36-907345.pdf" (id 3) (at 106.68 77.47 0)
+    (property "Datasheet" "https://www.mouser.com/datasheet/2/54/pvg5-907351.pdf" (id 3) (at 106.68 77.47 0)
       (effects (font (size 1.27 1.27)) hide)
     )
@@
       (effects (font (size 1.27 1.27)) (justify right))
     )
-    (property "Footprint" "LHRE Footprint Library:PV36W201C01B00" (id 2) (at 111.76 140.97 0)
+    (property "Footprint" "Global Libraries:PVG5A" (id 2) (at 111.76 140.97 0)
       (effects (font (size 1.27 1.27)) hide)
     )
-    (property "Datasheet" "https://www.mouser.com/datasheet/2/54/pv36-907345.pdf" (id 3) (at 111.76 140.97 0)
+    (property "Datasheet" "https://www.mouser.com/datasheet/2/54/pvg5-907351.pdf" (id 3) (at 111.76 140.97 0)
       (effects (font (size 1.27 1.27)) hide)
     )

Commit message: BSPD layout
Parts:
- renumbered U9 to U10
Changed lines of the file:
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@@
   (symbol (lib_id "Comparator:LM339") (at 71.12 92.71 0)
     (in_bom yes) (on_board yes)
-    (property "Reference" "U9" (id 0) (at 69.85 91.44 0)
+    (property "Reference" "U10" (id 0) (at 69.85 91.44 0)
       (effects (font (size 1.27 1.27)) (justify left))
     )
@@
       (effects (font (size 1.27 1.27)) hide)
     )
-    (pin "2")
-    (pin "4")
-    (pin "5")
+    (pin "12")
+    (pin "3")
   )
   (symbol (lib_id "power:+5V") (at 62.23 85.09 0)
@@
       (effects (font (size 1.27 1.27)) hide)
     )
-    (pin "2")
-    (pin "4")
-    (pin "5")
+    (pin "1")
+    (pin "6")
+    (pin "7")
   )
   (symbol (lib_id "power:+5V") (at 106.68 71.12 0)
@@
       (effects (font (size 1.27 1.27)) hide)
     )
-    (pin "2")
-    (pin "4")
-    (pin "5")
+    (pin "14")
+    (pin "8")
+    (pin "9")
   )
   (symbol (lib_id "Comparator:LM2901") (at 148.59 114.3 0)
@@
       (effects (font (size 1.27 1.27)) hide)
     )
-    (pin "2")
-    (pin "4")
-    (pin "5")
+    (pin "10")
+    (pin "11")
+    (pin "13")
   )
   (symbol (lib_id "power:+5V") (at 99.06 40.64 0)
