File: 23-BSPD-ELC/LDO.kicad_sch (KiCad schematic)
At the start: 0 parts

Commit message: Revision changes and updates to some footprints
Parts:
- added C38: 1uF, Capacitor_SMD:C_0603_1608Metric_Pad1.08x0.95mm_HandSolder, symbol Device:C
- added C39: 22uF, Capacitor_SMD:C_0603_1608Metric_Pad1.08x0.95mm_HandSolder, symbol Device:C
- added U20: AMS1117-3.3, Package_TO_SOT_SMD:SOT-223-3_TabPin2, symbol Regulator_Linear:AMS1117-3.3
Connections:
- new net 3v3_OUT: C39.1, U20.2 (VO)
- new net GND: C38.2, C39.2, U20.1 (GND)
- new net V_in: C38.1, U20.3 (VI)
Changed lines of the file:
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@@
 (kicad_sch (version 20211123) (generator eeschema)
   (paper "A4")
+  (junction (at 96.52 83.82) (diameter 0) (color 0 0 0 0)
+  )
+  (junction (at 123.19 83.82) (diameter 0) (color 0 0 0 0)
+  )
+  (wire (pts (xy 123.19 83.82) (xy 119.38 83.82))
+    (stroke (width 0) (type default) (color 0 0 0 0))
+  )
+  (wire (pts (xy 88.9 83.82) (xy 96.52 83.82))
+    (stroke (width 0) (type default) (color 0 0 0 0))
+  )
+  (wire (pts (xy 96.52 83.82) (xy 104.14 83.82))
+    (stroke (width 0) (type default) (color 0 0 0 0))
+  )
+  (wire (pts (xy 128.27 83.82) (xy 123.19 83.82))
+    (stroke (width 0) (type default) (color 0 0 0 0))
+  )
+  (hierarchical_label "V_in" (shape input) (at 88.9 83.82 180)
+    (effects (font (size 1.27 1.27)) (justify right))
+  )
+  (hierarchical_label "3v3_OUT" (shape output) (at 128.27 83.82 0)
+    (effects (font (size 1.27 1.27)) (justify left))
+  )
+  (symbol (lib_id "power:GND") (at 96.52 91.44 0) (unit 1)
+    (in_bom yes) (on_board yes) (fields_autoplaced)
+    (property "Reference" "#PWR0163" (id 0) (at 96.52 97.79 0)
+      (effects (font (size 1.27 1.27)) hide)
+    )
+    (property "Value" "GND" (id 1) (at 96.52 96.52 0))
+    (property "Footprint" "" (id 2) (at 96.52 91.44 0)
+      (effects (font (size 1.27 1.27)) hide)
+    )
+    (property "Datasheet" "" (id 3) (at 96.52 91.44 0)
+      (effects (font (size 1.27 1.27)) hide)
+    )
+    (pin "1")
+  )
+  (symbol (lib_id "Device:C") (at 123.19 87.63 0) (unit 1)
+    (in_bom yes) (on_board yes) (fields_autoplaced)
+    (property "Reference" "C39" (id 0) (at 127 86.3599 0)
+      (effects (font (size 1.27 1.27)) (justify left))
+    )
+    (property "Value" "22uF" (id 1) (at 127 88.8999 0)
+      (effects (font (size 1.27 1.27)) (justify left))
+    )
+    (property "Footprint" "Capacitor_SMD:C_0603_1608Metric_Pad1.08x0.95mm_HandSolder" (id 2) (at 124.1552 91.44 0)
+      (effects (font (size 1.27 1.27)) hide)
+    )
+    (property "Datasheet" "~" (id 3) (at 123.19 87.63 0)
+      (effects (font (size 1.27 1.27)) hide)
+    )
+    (pin "1")
+    (pin "2")
+  )
+  (symbol (lib_id "power:GND") (at 111.76 91.44 0) (unit 1)
+    (in_bom yes) (on_board yes) (fields_autoplaced)
+    (property "Reference" "#PWR0164" (id 0) (at 111.76 97.79 0)
+      (effects (font (size 1.27 1.27)) hide)
+    )
+    (property "Value" "GND" (id 1) (at 111.76 96.52 0))
+    (property "Footprint" "" (id 2) (at 111.76 91.44 0)
+      (effects (font (size 1.27 1.27)) hide)
+    )
+    (property "Datasheet" "" (id 3) (at 111.76 91.44 0)
+      (effects (font (size 1.27 1.27)) hide)
+    )
+    (pin "1")
+  )
+  (symbol (lib_id "power:GND") (at 123.19 91.44 0) (unit 1)
+    (in_bom yes) (on_board yes) (fields_autoplaced)
+    (property "Reference" "#PWR0165" (id 0) (at 123.19 97.79 0)
+      (effects (font (size 1.27 1.27)) hide)
+    )
+    (property "Value" "GND" (id 1) (at 123.19 96.52 0))
+    (property "Footprint" "" (id 2) (at 123.19 91.44 0)
+      (effects (font (size 1.27 1.27)) hide)
+    )
+    (property "Datasheet" "" (id 3) (at 123.19 91.44 0)
+      (effects (font (size 1.27 1.27)) hide)
+    )
+    (pin "1")
+  )
+  (symbol (lib_id "Device:C") (at 96.52 87.63 0) (unit 1)
+    (in_bom yes) (on_board yes) (fields_autoplaced)
+    (property "Reference" "C38" (id 0) (at 100.33 86.3599 0)
+      (effects (font (size 1.27 1.27)) (justify left))
+    )
+    (property "Value" "1uF" (id 1) (at 100.33 88.8999 0)
+      (effects (font (size 1.27 1.27)) (justify left))
+    )
+    (property "Footprint" "Capacitor_SMD:C_0603_1608Metric_Pad1.08x0.95mm_HandSolder" (id 2) (at 97.4852 91.44 0)
+      (effects (font (size 1.27 1.27)) hide)
+    )
+    (property "Datasheet" "~" (id 3) (at 96.52 87.63 0)
+      (effects (font (size 1.27 1.27)) hide)
+    )
+    (pin "1")
+    (pin "2")
+  )
+  (symbol (lib_id "Regulator_Linear:AMS1117-3.3") (at 111.76 83.82 0) (unit 1)
+    (in_bom yes) (on_board yes) (fields_autoplaced)
+    (property "Reference" "U20" (id 0) (at 111.76 76.2 0))
+    (property "Value" "AMS1117-3.3" (id 1) (at 111.76 78.74 0))
+    (property "Footprint" "Package_TO_SOT_SMD:SOT-223-3_TabPin2" (id 2) (at 111.76 78.74 0)
+      (effects (font (size 1.27 1.27)) hide)
+    )
+    (property "Datasheet" "http://www.advanced-monolithic.com/pdf/ds1117.pdf" (id 3) (at 114.3 90.17 0)
+      (effects (font (size 1.27 1.27)) hide)
+    )
+    (pin "1")
+    (pin "2")
+    (pin "3")
+  )
 )

Commit message: BSPD layout
Parts:
- renumbered C38 to C41, C39 to C42, U20 to U21
Changed lines of the file:
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@@
   (symbol (lib_id "power:GND") (at 96.52 91.44 0) (unit 1)
     (in_bom yes) (on_board yes) (fields_autoplaced)
-    (property "Reference" "#PWR0163" (id 0) (at 96.52 97.79 0)
+    (property "Reference" "#PWR0170" (id 0) (at 96.52 97.79 0)
       (effects (font (size 1.27 1.27)) hide)
     )
@@
   (symbol (lib_id "Device:C") (at 123.19 87.63 0) (unit 1)
     (in_bom yes) (on_board yes) (fields_autoplaced)
-    (property "Reference" "C39" (id 0) (at 127 86.3599 0)
+    (property "Reference" "C42" (id 0) (at 127 86.3599 0)
       (effects (font (size 1.27 1.27)) (justify left))
     )
@@
   (symbol (lib_id "power:GND") (at 111.76 91.44 0) (unit 1)
     (in_bom yes) (on_board yes) (fields_autoplaced)
-    (property "Reference" "#PWR0164" (id 0) (at 111.76 97.79 0)
+    (property "Reference" "#PWR0171" (id 0) (at 111.76 97.79 0)
       (effects (font (size 1.27 1.27)) hide)
     )
@@
   (symbol (lib_id "power:GND") (at 123.19 91.44 0) (unit 1)
     (in_bom yes) (on_board yes) (fields_autoplaced)
-    (property "Reference" "#PWR0165" (id 0) (at 123.19 97.79 0)
+    (property "Reference" "#PWR0172" (id 0) (at 123.19 97.79 0)
       (effects (font (size 1.27 1.27)) hide)
     )
@@
   (symbol (lib_id "Device:C") (at 96.52 87.63 0) (unit 1)
     (in_bom yes) (on_board yes) (fields_autoplaced)
-    (property "Reference" "C38" (id 0) (at 100.33 86.3599 0)
+    (property "Reference" "C41" (id 0) (at 100.33 86.3599 0)
       (effects (font (size 1.27 1.27)) (justify left))
     )
@@
   (symbol (lib_id "Regulator_Linear:AMS1117-3.3") (at 111.76 83.82 0) (unit 1)
     (in_bom yes) (on_board yes) (fields_autoplaced)
-    (property "Reference" "U20" (id 0) (at 111.76 76.2 0))
+    (property "Reference" "U21" (id 0) (at 111.76 76.2 0))
     (property "Value" "AMS1117-3.3" (id 1) (at 111.76 78.74 0))
     (property "Footprint" "Package_TO_SOT_SMD:SOT-223-3_TabPin2" (id 2) (at 111.76 78.74 0)
